Commit message: launch for controllers

File: my_robot_description/urdf/my_robot.ros2_control.xacro (robot description, xacro)
@@ -1,14 +1,19 @@
-<ros2_control name="MyRobotHWInterface" type="system">
-    <plugin>mock_component/GenericSystem</plugin>
-    <param name="calculate_dynamics">true</param>
-    <joint name="base_left_wheel_joint">
-        <command_interface name="velocity" />
-        <state_interface name="position" />
-        <state_interface name="velocity" />
-    </joint>
-    <joint name="base_right_wheel_joint">
-        <command_interface name="velocity" />
-        <state_interface name="position" />
-        <state_interface name="velocity" />
-    </joint>
-</ros2_control>
+<?xml version="1.0"?>
+<robot name="my_robot" xmlns:xacro="http://www.ros.org/wiki/xacro">
+    <ros2_control name="MyRobotHWInterface" type="system">
+        <hardware>
+            <plugin>mock_components/GenericSystem</plugin>
+            <param name="calculate_dynamics">true</param>
+        </hardware>
+        <joint name="base_left_wheel_joint">
+            <command_interface name="velocity" />
+            <state_interface name="position" />
+            <state_interface name="velocity" />
+        </joint>
+        <joint name="base_right_wheel_joint">
+            <command_interface name="velocity" />
+            <state_interface name="position" />
+            <state_interface name="velocity" />
+        </joint>
+    </ros2_control>
+</robot>

File: my_robot_description/urdf/my_robot.urdf.xacro (robot description, xacro)
@@ -3,3 +3,4 @@
     <xacro:include filename="materials.xacro" />
     <xacro:include filename="my_robot_core.xacro" />
+    <xacro:include filename="my_robot.ros2_control.xacro" />
 </robot>

File: my_robot_description/urdf/my_robot_core.xacro (robot description, xacro)
@@ -42,4 +42,5 @@
         <parent link="base_link" />
         <child link="left_wheel_link" />
+        <axis xyz="0 1 0"/>
     </joint>
     <link name="right_wheel_link">
@@ -57,4 +58,5 @@
         <parent link="base_link" />
         <child link="right_wheel_link" />
+        <axis xyz="0 1 0"/>
     </joint>
     <!-- Caster -->

Commit message: diff driver control manager working in gazebo, also FUCK THAT FUCKEN OUTDATED DOCUMENTATION FOR THIS FUCKEN SHIT

File: my_robot_description/urdf/my_robot.ros2_control.xacro (robot description, xacro)
@@ -1,8 +1,7 @@
 <?xml version="1.0"?>
 <robot name="my_robot" xmlns:xacro="http://www.ros.org/wiki/xacro">
-    <ros2_control name="MyRobotHWInterface" type="system">
+    <ros2_control name="GazeboSystem" type="system">
         <hardware>
-            <plugin>mock_components/GenericSystem</plugin>
-            <param name="calculate_dynamics">true</param>
+            <plugin>gz_ros2_control/GazeboSimSystem</plugin>
         </hardware>
         <joint name="base_left_wheel_joint">

File: my_robot_description/urdf/my_robot.urdf.xacro (robot description, xacro)
@@ -2,5 +2,7 @@
 <robot name="my_robot" xmlns:xacro="http://www.ros.org/wiki/xacro">
     <xacro:include filename="materials.xacro" />
+    <xacro:include filename="inertials.xacro" />
     <xacro:include filename="my_robot_core.xacro" />
+    <xacro:include filename="gz_plugins.xacro" />
     <xacro:include filename="my_robot.ros2_control.xacro" />
 </robot>

File: my_robot_description/urdf/my_robot_core.xacro (robot description, xacro)
@@ -4,9 +4,12 @@
     <xacro:property name="base_ly" value="0.15" />
     <xacro:property name="base_lz" value="0.05" />
+    <xacro:property name="base_mass" value="0.25" />
     <xacro:property name="wheel_rad" value="0.038" />
     <xacro:property name="wheel_len" value="0.026" />
+    <xacro:property name="wheel_mass" value="0.032" />
     <xacro:property name="base_wheel_offset_x" value="${base_lx * 0.3}" />
     <xacro:property name="base_wheel_offset_z" value="0" />
     <xacro:property name="caster_rad" value="0.02" />
+    <xacro:property name="caster_mass" value="0.07" />
     <xacro:property name="base_caster_offset_x" value="${base_lx * 0.4}" />
     <xacro:property name="base_caster_offset_z" value="${-base_lz * 0.5}" />
@@ -21,4 +24,12 @@
             <material name="red" />
         </visual>
+        <collision>
+            <origin xyz="0 0 0" rpy="0 0 0" />
+            <geometry>
+                <box size="${base_lx} ${base_ly} ${base_lz}" />
+            </geometry>
+        </collision>
+        <xacro:box_inertial lx="${base_lx}" ly="${base_ly}" lz="${base_lz}" m="${base_mass}"
+            o_xyz="0.0 0.0 0.0" o_rpy="0 0 0" />
     </link>
     <joint name="footprint_base_joint" type="fixed">
@@ -29,5 +40,5 @@
     <!-- Wheels -->
     <link name="left_wheel_link">
-        <visual name="">
+        <visual>
             <origin xyz="0.0 0.0 0.0" rpy="${pi/2} 0.0 0.0" />
             <geometry>
@@ -36,4 +47,12 @@
             <material name="black" />
         </visual>
+        <collision>
+            <origin xyz="0.0 0.0 0.0" rpy="${pi/2} 0.0 0.0" />
+            <geometry>
+                <cylinder radius="${wheel_rad}" length="${wheel_len}" />
+            </geometry>
+        </collision>
+        <xacro:cylinder_inertial r="${wheel_rad}" l="${wheel_len}" m="${wheel_mass}" o_xyz="0.0 0.0 0.0"
+            o_rpy="${pi/2} 0.0 0.0" />
     </link>
     <joint name="base_left_wheel_joint" type="continuous">
@@ -42,8 +61,8 @@
         <parent link="base_link" />
         <child link="left_wheel_link" />
-        <axis xyz="0 1 0"/>
+        <axis xyz="0 1 0" />
     </joint>
     <link name="right_wheel_link">
-        <visual name="">
+        <visual>
             <origin xyz="0.0 0.0 0.0" rpy="${pi/2} 0.0 0.0" />
             <geometry>
@@ -52,4 +71,12 @@
             <material name="black" />
         </visual>
+        <collision>
+            <origin xyz="0.0 0.0 0.0" rpy="${pi/2} 0.0 0.0" />
+            <geometry>
+                <cylinder radius="${wheel_rad}" length="${wheel_len}" />
+            </geometry>
+        </collision>
+        <xacro:cylinder_inertial r="${wheel_rad}" l="${wheel_len}" m="${wheel_mass}" o_xyz="0.0 0.0 0.0"
+            o_rpy="${pi/2} 0.0 0.0" />
     </link>
     <joint name="base_right_wheel_joint" type="continuous">
@@ -58,5 +85,5 @@
         <parent link="base_link" />
         <child link="right_wheel_link" />
-        <axis xyz="0 1 0"/>
+        <axis xyz="0 1 0" />
     </joint>
     <!-- Caster -->
@@ -69,9 +96,16 @@
             <material name="silver" />
         </visual>
+        <collision>
+            <origin xyz="0 0 ${-caster_rad / 2}" rpy="0 0 0" />
+            <geometry>
+                <sphere radius="${caster_rad}" />
+            </geometry>
+        </collision>
+        <xacro:sphere_inertial r="${caster_rad}" m="${caster_mass}" o_xyz="0 0 ${-caster_rad / 2}" o_rpy="0 0 0" />
     </link>
     <joint name="base_caster_joint" type="fixed">
-        <origin xyz="${base_caster_offset_x} 0 ${base_caster_offset_z}" rpy="0 0 0"/>
-        <parent link="base_link"/>
-        <child link="caster_link"/>
+        <origin xyz="${base_caster_offset_x} 0 ${base_caster_offset_z}" rpy="0 0 0" />
+        <parent link="base_link" />
+        <child link="caster_link" />
     </joint>
 </robot>
